Commit message: Update robot assets with new meshes and fix xacro paths
- Added updated mesh files with _1_1 suffixes
- Updated xacro file to use relative paths instead of ROS package paths
- Removed unused files and macOS metadata
- Maintained correct orientation (wheels up, springs down)

File: assets/jumping_robot_description_root/eecs4421_1d_hopper.urdf (robot description, URDF)
Before this commit: robot eecs4421_1d_hopper, 19 links, 18 joints
Links:
- removed link 2S_LiPo_1
- removed link 5x63mm_Aluminium_Rod__1_1
- removed link 5x63mm_Aluminium_Rod__2_1
- removed link Frame_V2_1
- removed link Main_Gear_1
- removed link Motor_1_1
- removed link Motor_2_1
- removed link Motor_Gear_1_1
- removed link Motor_Gear_2_1
- removed link Second_Gear_1
- removed link Servo_Gear_1
- removed link Servo_Pin_5x16mm_1
- removed link Spring_2_1
- removed link Spring__1
- removed link motor_1
- removed link moving_frame_1
- removed link wheel_1_complete_1
- removed link wheel_2_complete_1
- link base_link: mass 0.28240066077211035 -> 0.2824006607720704
Joints:
- removed joint 2S_LiPo_1_joint
- removed joint 5x63mm_Aluminium_Rod__1_1_joint
- removed joint 5x63mm_Aluminium_Rod__2_1_joint
- removed joint Frame_V2_1_joint
- removed joint Main_Gear_1_joint
- removed joint Motor_1_1_joint
- removed joint Motor_2_1_joint
- removed joint Motor_Gear_1_1_joint
- removed joint Motor_Gear_2_1_joint
- removed joint Second_Gear_1_joint
- removed joint Servo_Gear_1_joint
- removed joint Servo_Pin_5x16mm_1_joint
- removed joint Spring_2_1_joint
- removed joint Spring__1_joint
- removed joint motor_1_joint
- removed joint moving_frame_1_joint
- removed joint wheel_1_complete_1_joint
- removed joint wheel_2_complete_1_joint

File: assets/jumping_robot_description_root/urdf/jumping_robot_urdf_backup_copy.xacro (robot description, xacro)
@@ -6,6 +6,6 @@
 <link name="base_link">
   <inertial>
-    <origin xyz="-0.013572089715645304 0.07234958739791485 -0.0004353043515408574" rpy="0 0 0"/>
-    <mass value="0.28240066077211035"/>
+    <origin xyz="-0.013572090010166953 0.07234958657969306 -0.0004353043410476317" rpy="0 0 0"/>
+    <mass value="0.2824006607720704"/>
     <inertia ixx="0.001426" iyy="7.2e-05" izz="0.001359" ixy="-5e-06" iyz="-0.0" ixz="-0.0"/>
   </inertial>
